File: kicadproject/kicadproject.kicad_sch (KiCad schematic)
At the start: 0 parts

Commit message: add resistors
Parts:
- added R1, R2: R, symbol Device:R
Connections:
- new net: R1.2, R2.1
- new net GND: R1.1, R2.2
